Commit message: Task 2: xacro refactor into 5 macros + include_laser conditional

File: urdf/barista_robot_model.urdf (robot description, URDF)
Before this commit: robot barista_robot, 11 links, 10 joints
Links:
- link laser_scan_link: geometry collision cylinder length=0.040 radius=0.030; visual mesh filename=package://barista_robot_description/meshes/LASER_MESH.dae
